Commit message: Updates to the H1 config structure and retargeting script

File: phys_anim/data/assets/urdf/h1_no_head_no_hands.urdf (robot description, URDF)
Before this commit: robot h1, 23 links, 22 joints
Links:
- removed link head
- removed link left_arm_end_effector
- removed link right_arm_end_effector
Joints:
- removed joint head
- removed joint left_arm_end_effector_joint
- removed joint right_arm_end_effector_joint
